Commit message: Camera orientation fix.

File: source_code/ros_ws_robot_infra/src/ros_robot_description/urdf/components/rpi_camera.xacro (robot description, xacro)
@@ -18,5 +18,5 @@
         </link>
         <joint name="${name_prefix_fmt}camera_optical_joint" type="fixed">
-            <origin xyz="0 0 0" rpy="${-pi/2} 0 ${-pi/2}" />
+            <origin xyz="0 0 0" rpy="0 0 ${-pi/2}" />
             <parent link="${name_prefix_fmt}camera_link" />
             <child link="${name_prefix_fmt}camera_optical_link" />

Commit message: Camera orientation fix #2

File: source_code/ros_ws_robot_infra/src/ros_robot_description/urdf/components/rpi_camera.xacro (robot description, xacro)
@@ -18,5 +18,5 @@
         </link>
         <joint name="${name_prefix_fmt}camera_optical_joint" type="fixed">
-            <origin xyz="0 0 0" rpy="0 0 ${-pi/2}" />
+            <origin xyz="0 0 0" rpy="${-pi/2} 0 0" />
             <parent link="${name_prefix_fmt}camera_link" />
             <child link="${name_prefix_fmt}camera_optical_link" />

Commit message: Camera orientation fix #3

File: source_code/ros_ws_robot_infra/src/ros_robot_description/urdf/components/rpi_camera.xacro (robot description, xacro)
@@ -18,5 +18,5 @@
         </link>
         <joint name="${name_prefix_fmt}camera_optical_joint" type="fixed">
-            <origin xyz="0 0 0" rpy="${-pi/2} 0 0" />
+            <origin xyz="0 0 0" rpy="${pi/2} ${-pi/2} 0" />
             <parent link="${name_prefix_fmt}camera_link" />
             <child link="${name_prefix_fmt}camera_optical_link" />

Commit message: Fix camera flip.

File: source_code/ros_ws_robot_infra/src/ros_robot_description/urdf/components/rpi_camera.xacro (robot description, xacro)
@@ -17,7 +17,11 @@
             </visual>
         </link>
-        <xacro:property name="optical_frame_rot" value="${pi/2 if flip_optical else -pi/2}" />
         <joint name="${name_prefix_fmt}camera_optical_joint" type="fixed">
-            <origin xyz="0 0 0" rpy="${optical_frame_rot} 0 ${optical_frame_rot}" />
+            <xacro:if value="${flip_optical}">
+                <origin xyz="0 0 0" rpy="${pi/2} 0 ${pi/2}" />
+            </xacro:if>
+            <xacro:unless value="${flip_optical}">
+                <origin xyz="0 0 0" rpy="${-pi/2} 0 ${-pi/2}" />
+            </xacro:unless>
             <parent link="${name_prefix_fmt}camera_link" />
             <child link="${name_prefix_fmt}camera_optical_link" />
