Commit message: Robot description fixes, many new infra packages added. Ready for Nav2.

File: source_code/ros_ws_robot_infra/src/ros_robot_description/urdf/body.xacro (robot description, xacro)
@@ -1,19 +1,16 @@
 <?xml version="1.0" encoding="utf-8"?>
 <robot xmlns:xacro="http://www.ros.org/wiki/xacro">
-    <xacro:macro name="body" params="wheel_radius namespace">
+    <xacro:macro name="body" params="wheel_radius whl_z_offset namespace">
         <xacro:property name="body_mesh_file" value="package://ros_robot_description/meshes/robot_body.dae" />
         <xacro:property name="mass" value="2.2" />
-        <xacro:property name="inertia_ixx" value="0.01051" />
-        <xacro:property name="inertia_iyy" value="0.01893" />
-        <xacro:property name="inertia_izz" value="0.02458" />
         <xacro:property name="depth" value="0.3" />
         <xacro:property name="width" value="0.21" />
         <xacro:property name="height" value="0.115" />
-        <xacro:property name="camera_res" value="1280 720" />
-        <xacro:property name="camera_fps" value="20" />
         <xacro:property name="camera_fov" value="120" />
+        <xacro:property name="config_file" value="$(find ros_robot_description)/config/config.yaml" />
+        <xacro:property name="config" value="${xacro.load_yaml(config_file)}"/>
         <link name="base_link" />
-        <joint name="base_to_body_joint" type="fixed">
-            <origin xyz="0 0 ${wheel_radius}" rpy="0 0 0" />
+        <joint name="body_joint" type="fixed">
+            <origin xyz="0 0 ${wheel_radius-whl_z_offset}" rpy="0 0 0" />
             <parent link="base_link" />
             <child link="body_link" />
@@ -27,14 +24,12 @@
             </visual>
             <collision>
-                <!--<origin xyz="0 0 0" rpy="0 0 0" />-->
+                <origin xyz="0 0 ${height/2}" rpy="0 0 0" />
                 <geometry>
                     <box size="${depth} ${width} ${height}" />
                 </geometry>
             </collision>
-            <inertial>
-                <!--<origin xyz="0 0 0" rpy="0 0 0" />-->
-                <mass value="${mass}" />
-                <inertia ixx="${inertia_ixx}" iyy="${inertia_iyy}" izz="${inertia_izz}" />
-            </inertial>
+            <xacro:inertial_box mass="${mass}" x="${depth}" y="${width}" z="${height}">
+                <origin xyz="0 0 ${height/2}" rpy="0 0 0" />
+            </xacro:inertial_box>
         </link>
         <joint name="imu_joint" type="fixed">
@@ -51,5 +46,5 @@
         <xacro:camera_led parent_link="body_link" name_prefix="br" xyz="${cam_led_x} -0.018 0.06856" rpy="0 0 0" namespace="${namespace}" />
         <xacro:include filename="$(find ros_robot_description)/urdf/components/ir_cliff_sensor.xacro" />
-        <xacro:property name="cliff_sens_z" value="-0.01" />
+        <xacro:property name="cliff_sens_z" value="-0.0016" />
         <xacro:property name="cliff_sens_fx" value="${depth/2}" />
         <xacro:property name="cliff_sens_bx" value="${-depth/2}" />
@@ -69,14 +64,16 @@
         <xacro:micro_switch parent_link="body_link" name_prefix="br" xyz="${-micro_switch_x_ofst} -0.0898 ${micro_switch_z}" rpy="0 0 ${pi}" namespace="${namespace}" />
         <xacro:micro_switch parent_link="body_link" name_prefix="bl" xyz="${-micro_switch_x_ofst} 0.0898 ${micro_switch_z}" rpy="0 0 ${pi}" namespace="${namespace}" />
+        <xacro:property name="cam_config" value="${config['camera']}"/>
         <xacro:include filename="$(find ros_robot_description)/urdf/components/rpi_camera.xacro" />
-        <xacro:rpi_camera parent_link="body_link" xyz="${(depth/2)+0.01} 0 0.07856" rpy="0 0 0" namespace="${namespace}"
-                          fov="${camera_fov}" resolution="${camera_res}" fps="${camera_fps}" />
+        <xacro:rpi_camera parent_link="body_link" xyz="${(depth/2)+0.01} 0 0.09106" rpy="${pi} 0 0" namespace="${namespace}"
+                          resolution="${cam_config['simulation']['res_width']+' '+cam_config['simulation']['res_height']}"
+                          fps="${cam_config['simulation']['framerate']}" fov="${camera_fov}" />
         <xacro:include filename="$(find ros_robot_description)/urdf/components/rplidar_a1.xacro" />
-        <xacro:rplidar parent_link="body_link" name_prefix="lidar" xyz="0.08 0 ${height}" rpy="0 0 0" namespace="${namespace}" />
+        <xacro:rplidar parent_link="body_link" xyz="0.08 0 ${height}" rpy="0 0 0" namespace="${namespace}" />
         <xacro:include filename="$(find ros_robot_description)/urdf/components/ultrasonic.xacro" />
-        <xacro:ultrasonic type="srf05" parent_link="body_link" name_prefix="front" xyz="${(depth/2)-0.017} 0 0.03909" rpy="0 0 0" namespace="${namespace}" />
-        <xacro:ultrasonic type="hysrf05" parent_link="body_link" name_prefix="back" xyz="${(-depth/2)+0.0165} 0 0.03856" rpy="0 0 ${pi}" namespace="${namespace}" />
-        <xacro:ultrasonic type="hysrf05" parent_link="body_link" name_prefix="right" xyz="0 ${(-width/2)+0.0165} 0.07145" rpy="0 0 ${pi/2}" namespace="${namespace}" />
-        <xacro:ultrasonic type="hysrf05" parent_link="body_link" name_prefix="left" xyz="0 ${(width/2)-0.0165} 0.07145" rpy="0 0 ${-pi/2}" namespace="${namespace}" />
+        <xacro:ultrasonic type="srf05" parent_link="body_link" name_prefix="front" xyz="${(depth/2)-0.016} 0 0.03909" rpy="0 0 0" namespace="${namespace}" />
+        <xacro:ultrasonic type="hysrf05" parent_link="body_link" name_prefix="back" xyz="${(-depth/2)+0.0155} 0 0.03856" rpy="0 0 ${pi}" namespace="${namespace}" />
+        <xacro:ultrasonic type="hysrf05" parent_link="body_link" name_prefix="right" xyz="0 ${(-width/2)+0.0155} 0.07145" rpy="0 0 ${-pi/2}" namespace="${namespace}" />
+        <xacro:ultrasonic type="hysrf05" parent_link="body_link" name_prefix="left" xyz="0 ${(width/2)-0.0155} 0.07145" rpy="0 0 ${pi/2}" namespace="${namespace}" />
     </xacro:macro>
 </robot>

File: source_code/ros_ws_robot_infra/src/ros_robot_description/urdf/components/camera_led.xacro (robot description, xacro)
@@ -11,5 +11,4 @@
         <link name="${name_prefix}_cam_led_link">
             <visual>
-                <!-- <origin xyz="0 0 0" rpy="0 0 0" /> -->
                 <geometry>
                     <mesh filename="${mesh_file}" scale="1.0 1.0 1.0" />

File: source_code/ros_ws_robot_infra/src/ros_robot_description/urdf/components/ir_cliff_sensor.xacro (robot description, xacro)
@@ -4,4 +4,6 @@
         <xacro:property name="mesh_file" value="package://ros_robot_description/meshes/components/ir_cliff_sensor.dae" />
         <xacro:property name="namespace_fmt" value="${namespace + '/' if namespace != '' else ''}" />
+        <xacro:property name="component_config_file" value="$(find ros_robot_description)/config/components_config.yaml" />
+        <xacro:property name="component_config" value="${xacro.load_yaml(component_config_file)['ir_cliff_sensor']}"/>
         <joint name="${name_prefix}_cliff_sens_joint" type="fixed">
             <parent link="${parent_link}" />
@@ -11,5 +13,4 @@
         <link name="${name_prefix}_cliff_sens_link">
             <visual>
-                <origin xyz="${xyz}" rpy="${rpy}" />
                 <geometry>
                     <mesh filename="${mesh_file}" scale="1.0 1.0 1.0" />
@@ -20,5 +21,5 @@
             <sensor type="gpu_lidar" name="${namespace_fmt}${name_prefix}_cliff_sensor">
                 <pose>0 0 -0.003 ${-pi/2} 0 0</pose>
-                <update_rate>20</update_rate>
+                <update_rate>${component_config["simulation"]["update_rate"]}</update_rate>
                 <topic>${namespace_fmt}${name_prefix}_cliff_sensor/range</topic>
                 <gz_frame_id>${namespace_fmt}${name_prefix}_cliff_sens_link</gz_frame_id>

File: source_code/ros_ws_robot_infra/src/ros_robot_description/urdf/components/micro_switch.xacro (robot description, xacro)
@@ -4,4 +4,6 @@
         <xacro:property name="mesh_file" value="package://ros_robot_description/meshes/components/micro_switch.dae" />
         <xacro:property name="namespace_fmt" value="${namespace + '/' if namespace != '' else ''}" />
+        <xacro:property name="component_config_file" value="$(find ros_robot_description)/config/components_config.yaml" />
+        <xacro:property name="component_config" value="${xacro.load_yaml(component_config_file)['micro_switch']}"/>
         <joint name="${name_prefix}_microswitch_joint" type="fixed">
             <parent link="${parent_link}" />
@@ -11,5 +13,4 @@
         <link name="${name_prefix}_microswitch_link">
             <visual>
-                <origin xyz="${xyz}" rpy="${rpy}" />
                 <geometry>
                     <mesh filename="${mesh_file}" scale="1.0 1.0 1.0" />
@@ -17,5 +18,5 @@
             </visual>
             <collision name="${name_prefix}_microswitch_collision">
-                <origin xyz="0.004" rpy="0 0 0" />
+                <origin xyz="0.004 0 0" rpy="0 0 0" />
                 <geometry>
                     <box size="0.018 0.006 0.02"/>
@@ -25,5 +26,5 @@
         <gazebo reference="${name_prefix}_microswitch_link">
             <sensor type="contact" name="${namespace_fmt}${name_prefix}_microswitch_sensor">
-                <update_rate>50</update_rate>
+                <update_rate>${component_config["simulation"]["update_rate"]}</update_rate>
                 <topic>${namespace_fmt}${name_prefix}_microswitch/contact</topic>
                 <gz_frame_id>${namespace_fmt}${name_prefix}_microswitch_link</gz_frame_id>

File: source_code/ros_ws_robot_infra/src/ros_robot_description/urdf/components/rpi_camera.xacro (robot description, xacro)
@@ -22,5 +22,5 @@
             <child link="${name_prefix_fmt}camera_optical_link" />
         </joint>
-        <link name="${name_prefix_fmt}camera_optical_link"></link>
+        <link name="${name_prefix_fmt}camera_optical_link" />
         <gazebo reference="${name_prefix_fmt}camera_link">
             <sensor type="camera" name="${namespace_fmt}${name_prefix_fmt}camera">

File: source_code/ros_ws_robot_infra/src/ros_robot_description/urdf/components/rplidar_a1.xacro (robot description, xacro)
@@ -1,15 +1,16 @@
 <?xml version="1.0" encoding="utf-8"?>
 <robot xmlns:xacro="http://www.ros.org/wiki/xacro">
-    <xacro:macro name="rplidar" params="parent_link name_prefix namespace xyz rpy">
+    <xacro:macro name="rplidar" params="parent_link name_prefix:='' namespace xyz rpy">
         <xacro:property name="namespace_fmt" value="${namespace + '/' if namespace != '' else ''}" />
+        <xacro:property name="name_prefix_fmt" value="${name_prefix + '_' if name_prefix != '' else ''}" />
+        <xacro:property name="component_config_file" value="$(find ros_robot_description)/config/components_config.yaml" />
+        <xacro:property name="component_config" value="${xacro.load_yaml(component_config_file)['rplidar']}"/>
         <xacro:property name="mass" value="0.190" />
-        <xacro:property name="inertia_ixx" value="0.00010608" />
-        <xacro:property name="inertia_iyy" value="0.00010608" />
-        <xacro:property name="inertia_izz" value="0.00011638" />
         <xacro:property name="radius" value="0.035" />
         <xacro:property name="height" value="0.055" />
-        <joint name="${name_prefix}_laser_joint" type="fixed">
+        <xacro:property name="sensor_dist_from_top" value="0.008" />
+        <joint name="${name_prefix_fmt}lidar_joint" type="fixed">
             <parent link="${parent_link}" />
-            <child link="${name_prefix}_laser_link" />
+            <child link="${name_prefix_fmt}lidar_link" />
             <origin xyz="${xyz}" rpy="${rpy}" />
         </joint>
@@ -20,5 +21,5 @@
             </geometry>
         </xacro:property>
-        <link name="${name_prefix}_laser_link">
+        <link name="${name_prefix_fmt}lidar_link">
             <visual>
                 <!-- No proper Collada mesh for the RPLiDAR-A1M8 yet -->
@@ -29,16 +30,22 @@
                 <xacro:insert_block name="collision_mesh" />
             </collision>
-            <inertial>
-                <mass value="${mass}" />
-                <inertia ixx="${inertia_ixx}" iyy="${inertia_iyy}" izz="${inertia_izz}" />
-            </inertial>
+            <xacro:inertial_cylinder mass="${mass}" length="${height}" radius="${radius}">
+                <origin xyz="0 0 0" rpy="0 0 0"/>
+            </xacro:inertial_cylinder>
         </link>
-        <gazebo reference="${name_prefix}_laser_link">
+        <joint name="${name_prefix_fmt}lidar_laser_joint" type="fixed">
+            <origin xyz="0 0 ${height-sensor_dist_from_top}" rpy="0 0 0" />
+            <parent link="${name_prefix_fmt}lidar_link" />
+            <child link="${name_prefix_fmt}lidar_laser_link" />
+        </joint>
+        <link name="${name_prefix_fmt}lidar_laser_link" />
+        <gazebo reference="${name_prefix_fmt}lidar_link">
             <material>Gazebo/Red</material>
             <sensor type="gpu_lidar" name="${namespace_fmt}${name_prefix}_laser_sensor">
+                <pose>0 0 ${height-sensor_dist_from_top} 0 0 0</pose>
                 <visualize>false</visualize>
-                <update_rate>10</update_rate>
-                <topic>${namespace_fmt}${name_prefix}_laser/scan</topic>
-                <gz_frame_id>${namespace_fmt}${name_prefix}_laser_link</gz_frame_id>
+                <update_rate>${component_config["simulation"]["update_rate"]}</update_rate>
+                <topic>${namespace_fmt}${name_prefix_fmt}lidar/scan</topic>
+                <gz_frame_id>${namespace_fmt}${name_prefix_fmt}lidar_laser_link</gz_frame_id>
                 <lidar>
                     <scan>

File: source_code/ros_ws_robot_infra/src/ros_robot_description/urdf/components/ultrasonic.xacro (robot description, xacro)
@@ -4,4 +4,6 @@
         <xacro:property name="namespace_fmt" value="${namespace + '/' if namespace != '' else ''}" />
         <xacro:property name="mesh_file" value="package://ros_robot_description/meshes/components/ultrasonic_${type}.dae" />
+        <xacro:property name="component_config_file" value="$(find ros_robot_description)/config/components_config.yaml" />
+        <xacro:property name="component_config" value="${xacro.load_yaml(component_config_file)['ultrasonic']}"/>
         <xacro:if value="${type == 'hysrf05'}">
             <xacro:property name="min_meas_dist" value="0.02" />
@@ -27,5 +29,4 @@
         <link name="${name_prefix}_ultrasonic_link">
             <visual>
-                <origin xyz="${xyz}" rpy="${rpy}" />
                 <geometry>
                     <mesh filename="${mesh_file}" scale="1.0 1.0 1.0" />
@@ -33,10 +34,16 @@
             </visual>
         </link>
+        <joint name="${name_prefix}_ultrasonic_emit_joint" type="fixed">
+            <origin xyz="${sens_x_offset} 0 0" rpy="0 0 0" />
+            <parent link="${name_prefix}_ultrasonic_link" />
+            <child link="${name_prefix}_ultrasonic_emit_link" />
+        </joint>
+        <link name="${name_prefix}_ultrasonic_emit_link" />
         <gazebo reference="${name_prefix}_ultrasonic_link">
             <sensor type="gpu_lidar" name="${namespace_fmt}${name_prefix}_ultrasonic_sensor">
                 <pose>${sens_x_offset} 0 0 0 0 0</pose>
-                <update_rate>10</update_rate>
+                <update_rate>${component_config["simulation"]["update_rate"]}</update_rate>
                 <topic>${namespace_fmt}${name_prefix}_ultrasonic/range</topic>
-                <gz_frame_id>${namespace_fmt}${name_prefix}_ultrasonic_link</gz_frame_id>
+                <gz_frame_id>${namespace_fmt}${name_prefix}_ultrasonic_emit_link</gz_frame_id>
                 <visualize>false</visualize>
                 <lidar>
@@ -60,7 +67,5 @@
                         <resolution>${meas_res}</resolution>
                     </range>
-                    <noise type="gaussian">
-                        <stddev>${gauss_std_dev}</stddev>
-                    </noise>
+                    <xacro:gaussian_noise stddev="${gauss_std_dev}" />
                 </lidar>
             </sensor>

File: source_code/ros_ws_robot_infra/src/ros_robot_description/urdf/gazebo.xacro (robot description, xacro)
@@ -1,19 +1,13 @@
 <?xml version="1.0" encoding="utf-8"?>
 <robot xmlns:xacro="http://wiki.ros.org/xacro">
+    <xacro:include filename="$(find ros_robot_description)/urdf/utils/common_macros.xacro" />
     <!-- Noise values are for the MPU6050 -->
     <xacro:macro name="imu" params="reference_frame namespace:=''">
         <xacro:property name="namespace_fmt" value="${namespace + '/' if namespace != '' else ''}" />
-        <xacro:macro name="gaussian_noise" params="stddev bias_mean:=0 bias_stddev:=0 precision:=0 mean:=0">
-            <noise type="gaussian">
-                <stddev>${stddev}</stddev>
-                <bias_mean>${bias_mean}</bias_mean>
-                <bias_stddev>${bias_stddev}</bias_stddev>
-                <precision>${precision}</precision>
-                <mean>${mean}</mean>
-            </noise>
-        </xacro:macro>
+        <xacro:property name="config_file" value="$(find ros_robot_description)/config/config.yaml" />
+        <xacro:property name="config" value="${xacro.load_yaml(config_file)['imu']['simulation']}"/>
         <gazebo reference="${reference_frame}">
             <sensor name="${namespace_fmt}imu" type="imu">
-                <update_rate>20</update_rate>
+                <update_rate>${config["update_rate"]}</update_rate>
                 <topic>${namespace_fmt}imu/data_raw</topic>
                 <gz_frame_id>${namespace_fmt}imu_link</gz_frame_id>

File: source_code/ros_ws_robot_infra/src/ros_robot_description/urdf/ros_robot.urdf.xacro (robot description, xacro)
@@ -3,17 +3,19 @@
     <xacro:arg name="namespace" default="" />
     <xacro:arg name="use_sim" default="false" />
+    <xacro:property name="wheel_shaft_z_offset" value="0.02" />
     <xacro:property name="wheel_radius" value="0.05" />
     <xacro:property name="wheel_thickness" value="0.015" />
     <xacro:property name="track_width" value="0.25" />
     <xacro:property name="wheelbase" value="0.14" />
-    <xacro:include filename="$(find ros_robot_description)/urdf/materials.xacro" />
+    <xacro:include filename="$(find ros_robot_description)/urdf/utils/materials.xacro" />
+    <xacro:include filename="$(find ros_robot_description)/urdf/utils/common_macros.xacro" />
     <xacro:include filename="$(find ros_robot_description)/urdf/gazebo.xacro" ns="gazebo" />
     <xacro:include filename="$(find ros_robot_description)/urdf/body.xacro" />
     <xacro:include filename="$(find ros_robot_description)/urdf/wheel.xacro" />
-    <xacro:body wheel_radius="${wheel_radius}" namespace="$(arg namespace)" />
-    <xacro:wheel position="fr" wheel_radius="${wheel_radius}" wheel_thickness="${wheel_thickness}" wheelbase="${wheelbase}" track_width="${track_width}" />
-    <xacro:wheel position="fl" wheel_radius="${wheel_radius}" wheel_thickness="${wheel_thickness}" wheelbase="${wheelbase}" track_width="${track_width}" />
-    <xacro:wheel position="br" wheel_radius="${wheel_radius}" wheel_thickness="${wheel_thickness}" wheelbase="${wheelbase}" track_width="${track_width}" />
-    <xacro:wheel position="bl" wheel_radius="${wheel_radius}" wheel_thickness="${wheel_thickness}" wheelbase="${wheelbase}" track_width="${track_width}" />
+    <xacro:body wheel_radius="${wheel_radius}" whl_z_offset="${wheel_shaft_z_offset}" namespace="$(arg namespace)" />
+    <xacro:wheel position="fr" wheel_radius="${wheel_radius}" wheel_thickness="${wheel_thickness}" wheelbase="${wheelbase}" track_width="${track_width}" whl_z_offset="${wheel_shaft_z_offset}" />
+    <xacro:wheel position="fl" wheel_radius="${wheel_radius}" wheel_thickness="${wheel_thickness}" wheelbase="${wheelbase}" track_width="${track_width}" whl_z_offset="${wheel_shaft_z_offset}" />
+    <xacro:wheel position="br" wheel_radius="${wheel_radius}" wheel_thickness="${wheel_thickness}" wheelbase="${wheelbase}" track_width="${track_width}" whl_z_offset="${wheel_shaft_z_offset}" />
+    <xacro:wheel position="bl" wheel_radius="${wheel_radius}" wheel_thickness="${wheel_thickness}" wheelbase="${wheelbase}" track_width="${track_width}" whl_z_offset="${wheel_shaft_z_offset}" />
     <xacro:unless value="$(arg use_sim)">
     </xacro:unless>
