Commit message: Robot description fixes, many new infra packages added. Ready for Nav2.

File: source_code/ros_ws_robot_infra/src/ros_robot_description/urdf/wheel.xacro (robot description, xacro)
@@ -1,34 +1,31 @@
 <?xml version="1.0" encoding="utf-8"?>
 <robot xmlns:xacro="http://www.ros.org/wiki/xacro">
-    <xacro:macro name="wheel" params="position wheel_radius wheel_thickness wheelbase track_width">
+    <xacro:macro name="wheel" params="position wheel_radius wheel_thickness wheelbase track_width whl_z_offset">
         <xacro:property name="mesh_file" value="package://ros_robot_description/meshes/robot_wheel.dae" />
         <xacro:property name="mass" value="0.036" />
-        <xacro:property name="inertia_ixx" value="0.000024" />
-        <xacro:property name="inertia_iyy" value="0.000046" />
-        <xacro:property name="inertia_izz" value="0.000024" />
         <xacro:if value="${position == 'fr'}">
             <xacro:property name="pos_x" value="${wheelbase/2.0}" />
             <xacro:property name="pos_y" value="${-track_width/2.0}" />
-            <xacro:property name="mesh_yaw" value="${pi}" />
+            <xacro:property name="mesh_roll" value="${pi/2}" />
         </xacro:if>
         <xacro:if value="${position == 'fl'}">
             <xacro:property name="pos_x" value="${wheelbase/2.0}" />
             <xacro:property name="pos_y" value="${track_width/2.0}" />
-            <xacro:property name="mesh_yaw" value="0" />
+            <xacro:property name="mesh_roll" value="${-pi/2}" />
         </xacro:if>
         <xacro:if value="${position == 'br'}">
             <xacro:property name="pos_x" value="${-wheelbase/2.0}" />
             <xacro:property name="pos_y" value="${-track_width/2.0}" />
-            <xacro:property name="mesh_yaw" value="${pi}" />
+            <xacro:property name="mesh_roll" value="${pi/2}" />
         </xacro:if>
         <xacro:if value="${position == 'bl'}">
             <xacro:property name="pos_x" value="${-wheelbase/2.0}" />
             <xacro:property name="pos_y" value="${track_width/2.0}" />
-            <xacro:property name="mesh_yaw" value="0" />
+            <xacro:property name="mesh_roll" value="${-pi/2}" />
         </xacro:if>
         <joint name="${position}_wheel_joint" type="continuous">
             <parent link="body_link" />
             <child link="${position}_wheel_link" />
-            <origin xyz="${pos_x} ${pos_y} 0" rpy="0 0 0" />
+            <origin xyz="${pos_x} ${pos_y} ${whl_z_offset}" rpy="${pi/2} 0 0" />
             <axis xyz="0 1.0 0" />
             <limit effort="1.5" velocity="0.62" />
@@ -37,5 +34,5 @@
         <link name="${position}_wheel_link">
             <visual>
-                <origin xyz="0 0 0" rpy="0 0 ${mesh_yaw}" />
+                <origin xyz="0 0 0" rpy="${mesh_roll} 0 0" />
                 <geometry>
                     <mesh filename="${mesh_file}" scale="1.0 1.0 1.0" />
@@ -43,13 +40,11 @@
             </visual>
             <collision>
-                <origin xyz="0 0 0" rpy="${pi/2} 0 0" />
                 <geometry>
                     <cylinder radius="${wheel_radius}" length="${wheel_thickness}" />
                 </geometry>
             </collision>
-            <inertial>
-                <mass value="${mass}" />
-                <inertia ixx="${inertia_ixx}" iyy="${inertia_iyy}" izz="${inertia_izz}" />
-            </inertial>
+            <xacro:inertial_cylinder mass="${mass}" length="${wheel_thickness}" radius="${wheel_radius}">
+                <origin xyz="0 0 0" rpy="0 0 0"/>
+            </xacro:inertial_cylinder>
         </link>
         <gazebo reference="${position}_wheel_link">

Commit message: Fixed camera (optical) orientation.

File: source_code/ros_ws_robot_infra/src/ros_robot_description/urdf/body.xacro (robot description, xacro)
@@ -66,5 +66,5 @@
         <xacro:property name="cam_config" value="${config['camera']}"/>
         <xacro:include filename="$(find ros_robot_description)/urdf/components/rpi_camera.xacro" />
-        <xacro:rpi_camera parent_link="body_link" xyz="${(depth/2)+0.01} 0 0.09106" rpy="${pi} 0 0" namespace="${namespace}"
+        <xacro:rpi_camera parent_link="body_link" xyz="${(depth/2)+0.01} 0 0.09106" rpy="${pi} 0 0" flip_optical="True" namespace="${namespace}"
                           resolution="${cam_config['simulation']['res_width']+' '+cam_config['simulation']['res_height']}"
                           fps="${cam_config['simulation']['framerate']}" fov="${camera_fov}" />

File: source_code/ros_ws_robot_infra/src/ros_robot_description/urdf/components/rpi_camera.xacro (robot description, xacro)
@@ -1,5 +1,5 @@
 <?xml version="1.0" encoding="utf-8"?>
 <robot xmlns:xacro="http://www.ros.org/wiki/xacro">
-    <xacro:macro name="rpi_camera" params="parent_link name_prefix:='' namespace xyz rpy fov resolution fps">
+    <xacro:macro name="rpi_camera" params="parent_link name_prefix:='' namespace xyz rpy flip_optical:=False fov resolution fps">
         <xacro:property name="mesh_file" value="package://ros_robot_description/meshes/components/rpi_camera.dae" />
         <xacro:property name="namespace_fmt" value="${namespace + '/' if namespace != '' else ''}" />
@@ -17,6 +17,7 @@
             </visual>
         </link>
+        <xacro:property name="optical_frame_rot" value="${pi/2 if flip_optical else -pi/2}" />
         <joint name="${name_prefix_fmt}camera_optical_joint" type="fixed">
-            <origin xyz="0 0 0" rpy="${pi/2} ${-pi/2} 0" />
+            <origin xyz="0 0 0" rpy="${optical_frame_rot} 0 ${optical_frame_rot}" />
             <parent link="${name_prefix_fmt}camera_link" />
             <child link="${name_prefix_fmt}camera_optical_link" />

Commit message: Fixed wheel rotation axis.

File: source_code/ros_ws_robot_infra/src/ros_robot_description/urdf/body.xacro (robot description, xacro)
@@ -60,8 +60,8 @@
         <xacro:property name="micro_switch_z" value="0.01811" />
         <xacro:property name="micro_switch_x_ofst" value="${(depth/2)-0.005}" />
-        <xacro:micro_switch parent_link="body_link" name_prefix="fr" xyz="${micro_switch_x_ofst} -0.0898 ${micro_switch_z}" rpy="0 0 0" namespace="${namespace}" />
-        <xacro:micro_switch parent_link="body_link" name_prefix="fl" xyz="${micro_switch_x_ofst} 0.0898 ${micro_switch_z}" rpy="0 0 0" namespace="${namespace}" />
-        <xacro:micro_switch parent_link="body_link" name_prefix="br" xyz="${-micro_switch_x_ofst} -0.0898 ${micro_switch_z}" rpy="0 0 ${pi}" namespace="${namespace}" />
-        <xacro:micro_switch parent_link="body_link" name_prefix="bl" xyz="${-micro_switch_x_ofst} 0.0898 ${micro_switch_z}" rpy="0 0 ${pi}" namespace="${namespace}" />
+        <xacro:micro_switch parent_link="body_link" name_prefix="front_right" xyz="${micro_switch_x_ofst} -0.0898 ${micro_switch_z}" rpy="0 0 0" namespace="${namespace}" />
+        <xacro:micro_switch parent_link="body_link" name_prefix="front_left" xyz="${micro_switch_x_ofst} 0.0898 ${micro_switch_z}" rpy="0 0 0" namespace="${namespace}" />
+        <xacro:micro_switch parent_link="body_link" name_prefix="back_right" xyz="${-micro_switch_x_ofst} -0.0898 ${micro_switch_z}" rpy="0 0 ${pi}" namespace="${namespace}" />
+        <xacro:micro_switch parent_link="body_link" name_prefix="back_left" xyz="${-micro_switch_x_ofst} 0.0898 ${micro_switch_z}" rpy="0 0 ${pi}" namespace="${namespace}" />
         <xacro:property name="cam_config" value="${config['camera']}"/>
         <xacro:include filename="$(find ros_robot_description)/urdf/components/rpi_camera.xacro" />

File: source_code/ros_ws_robot_infra/src/ros_robot_description/urdf/wheel.xacro (robot description, xacro)
@@ -28,5 +28,5 @@
             <child link="${position}_wheel_link" />
             <origin xyz="${pos_x} ${pos_y} ${whl_z_offset}" rpy="${pi/2} 0 0" />
-            <axis xyz="0 1.0 0" />
+            <axis xyz="0 0 1" />
             <limit effort="1.5" velocity="0.62" />
             <dynamics damping="0.001" friction="0.001" />
